Commit message: updated

File: src/r2d2/urdf/myrobot1.urdf (robot description, URDF)
Before this commit: robot my_robot, 16 links, 15 joints
Joints:
- removed joint left_wheel_hinge
- removed joint right_wheel_hinge
- added joint left_wheel: type revolute, parent base_link, child left_wheel, origin xyz=-.29 -.17 -.155 rpy=0 1.5707 0, axis 0 0 0, limit lower=0 upper=6.28 effort=4 velocity=10
- added joint right_wheel: type revolute, parent base_link, child right_wheel, origin xyz=0.29 -.17 -.155 rpy=0 1.5707 0, axis 0 0 0, limit lower=0 upper=6.28 effort=4 velocity=10
- joint camera_depth_joint: origin xyz=0 0 0 rpy=0 0 0 -> xyz=0 0 0 rpy=0 0 2.35
- joint camera_depth_optical_joint: origin xyz=0 0 0 rpy=0 0 0 -> xyz=0 0 0 rpy=0 0 2.35
- joint camera_rgb_joint: origin xyz=-0.09 0 0.25 rpy=0 0 0 -> xyz=-0.09 0 0.25 rpy=0 0 2.35
- joint camera_rgb_optical_joint: origin xyz=0 0 0 rpy=0 0 0 -> xyz=0 0 0 rpy=0 0 2.35
